File: PCB/pihat_cooling.kicad_pcb (KiCad board)
At the start: 2 copper layers, 65 x 56 mm, 10 parts, among them M1 Fan, P1 Conn_02x20_Odd_Even

Commit message: fix sch + add more 3d model
Parts:
- added C1: CP, Capacitor_THT:CP_Radial_D7.5mm_P2.50mm, F.Cu at (365.0, 129.9)
- added C2: CP, Capacitor_THT:CP_Radial_D7.5mm_P2.50mm, F.Cu at (336.0, 145.7)
- added C3: CP, Capacitor_THT:CP_Radial_D7.5mm_P2.50mm, F.Cu at (345.2, 141.6)
- added C4: CP, Capacitor_THT:CP_Radial_D7.5mm_P2.50mm, F.Cu at (355.8, 138.9)
- added D1: 5V1, Diode_THT:D_DO-35_SOD27_P7.62mm_Horizontal, F.Cu at (320.2, 147.2)
- added D10: LD_5V, Displays:LED_D3.0mm, F.Cu at (376.8, 118.2)
- added D11: D4148, Diode_THT:D_DO-41_SOD81_P10.16mm_Horizontal, F.Cu at (306.6, 141.6)
- added D12: 1N4007, Diode_THT:D_DO-41_SOD81_P10.16mm_Horizontal, F.Cu at (352.5, 119.0)
- added D2: 1N4007, Diode_THT:D_DO-41_SOD81_P10.16mm_Horizontal, F.Cu at (306.6, 145.9)
- added D3: 1N4007, Diode_THT:D_DO-41_SOD81_P10.16mm_Horizontal, F.Cu at (306.6, 137.4)
- added D4: 1N4007, Diode_THT:D_DO-41_SOD81_P10.16mm_Horizontal, F.Cu at (320.5, 143.3)
- added D5: 1N4007, Diode_THT:D_DO-41_SOD81_P10.16mm_Horizontal, F.Cu at (370.2, 106.6)
- added D6: 5V1, Diode_THT:D_DO-35_SOD27_P7.62mm_Horizontal, F.Cu at (352.2, 122.9)
- added D7: 1N5820, Diode_THT:D_DO-201AD_P15.24mm_Horizontal, F.Cu at (307.1, 131.9)
- added D8: LD_Thermal, Displays:LED_D3.0mm, F.Cu at (320.3, 138.0)
- added D9: LED_12V, Displays:LED_D3.0mm, F.Cu at (378.4, 111.5)
- added J1: Barrel_Jack, Connector_BarrelJack:BarrelJack_Horizontal, F.Cu at (339.2, 133.9)
- added J2: Conn_01x03, Connector_PinHeader_2.54mm:PinHeader_1x03_P2.54mm_Vertical, F.Cu at (354.6, 127.0)
- added L1: 33uF, Inductor_SMD:L_Vishay_IHLP-2020, F.Cu at (372.5, 112.1)
- added Q1: AO3401A, Package_TO_SOT_SMD:SOT-23, F.Cu at (359.2, 126.9)
- added Q2: MMBT3906, Package_TO_SOT_SMD:SOT-23, F.Cu at (359.2, 131.5)
- added Q3: AO3401A, Package_TO_SOT_SMD:SOT-23, F.Cu at (363.7, 139.7)
- added Q4: MMBT3904, Package_TO_SOT_SMD:SOT-23, F.Cu at (373.0, 130.6)
- added R1: 100K, Resistor_SMD:R_0805_2012Metric_Pad1.15x1.40mm_HandSolder, F.Cu at (353.6, 147.8)
- added R10: 100, Resistor_SMD:R_0805_2012Metric_Pad1.15x1.40mm_HandSolder, F.Cu at (344.1, 147.6)
- added R2: 2K2, Resistor_SMD:R_0805_2012Metric_Pad1.15x1.40mm_HandSolder, F.Cu at (358.1, 144.9)
- added R3: 1K, Resistor_SMD:R_0805_2012Metric_Pad1.15x1.40mm_HandSolder, F.Cu at (348.9, 147.8)
- added R4: 100K, Resistor_SMD:R_0805_2012Metric_Pad1.15x1.40mm_HandSolder, F.Cu at (383.4, 115.8)
- added R5: 1K, Resistor_SMD:R_0805_2012Metric_Pad1.15x1.40mm_HandSolder, F.Cu at (377.5, 122.4)
- added R6: 1K, Resistor_SMD:R_0805_2012Metric_Pad1.15x1.40mm_HandSolder, F.Cu at (373.1, 126.9)
- added R7: 1K, Resistor_SMD:R_0805_2012Metric_Pad1.15x1.40mm_HandSolder, F.Cu at (363.9, 135.9)
- added R8: 100, Resistor_SMD:R_0805_2012Metric_Pad1.15x1.40mm_HandSolder, F.Cu at (383.4, 118.7)
- added R9: 100, Resistor_SMD:R_0805_2012Metric_Pad1.15x1.40mm_HandSolder, F.Cu at (353.3, 144.9)
- added SW1: Shutdown, Button_Switch_THT:SW_PUSH_6mm, F.Cu at (343.8, 130.5)
- added SW2: Reboot, Button_Switch_THT:SW_PUSH_6mm, F.Cu at (366.6, 118.9)
- added TP1: TestPoint, TestPoint:TestPoint_Pad_D1.0mm, F.Cu at (363.0, 122.6)
- added TP2: TestPoint, TestPoint:TestPoint_Pad_D1.0mm, F.Cu at (383.8, 106.0)
- added TP3: TestPoint, TestPoint:TestPoint_Pad_D1.0mm, F.Cu at (330.9, 146.9)
- added U1: LM2596S-5, Package_TO_SOT_SMD:TO-263-5_TabPin3, F.Cu at (359.5, 110.7)
- added U2: DS3231_RTC_Module, pihat_cooling:DS3231_RTC_Module, B.Cu at (186.2, 130.3)
Connections:
- net +5V renamed +5VP
- P1 pad 10: /GPIO15(RXD0) -> (no net)
- P1 pad 11: /GPIO17(GEN0) -> /Thermal_Pin
- P1 pad 12: /GPIO18(GEN1)(PWM0) -> /PWM_Pin
- P1 pad 13: /GPIO27(GEN2) -> /Shutdown_Pin
- P1 pad 15: /GPIO22(GEN3) -> /Reboot_Pin
- P1 pad 16: /GPIO23(GEN4) -> (no net)
- P1 pad 18: /GPIO24(GEN5) -> (no net)
- P1 pad 19: /GPIO10(SPI0_MOSI) -> (no net)
- P1 pad 21: /GPIO9(SPI0_MISO) -> (no net)
- P1 pad 22: /GPIO25(GEN6) -> (no net)
- P1 pad 23: /GPIO11(SPI0_SCK) -> (no net)
- P1 pad 24: /GPIO8(SPI0_CE_N) -> (no net)
- P1 pad 26: /GPIO7(SPI1_CE_N) -> (no net)
- P1 pad 27: /ID_SD -> (no net)
- P1 pad 28: /ID_SC -> (no net)
- P1 pad 29: /GPIO5 -> (no net)
- P1 pad 3: /GPIO2(SDA1) -> (no net)
- P1 pad 31: /GPIO6 -> (no net)
- P1 pad 32: /GPIO12(PWM0) -> (no net)
- P1 pad 33: /GPIO13(PWM1) -> (no net)
- P1 pad 35: /GPIO19(SPI1_MISO) -> (no net)
- P1 pad 36: /GPIO16 -> (no net)
- P1 pad 37: /GPIO26 -> (no net)
- P1 pad 38: /GPIO20(SPI1_MOSI) -> (no net)
- P1 pad 40: /GPIO21(SPI1_SCK) -> (no net)
- P1 pad 5: /GPIO3(SCL1) -> (no net)
- P1 pad 7: /GPIO4(GCLK) -> (no net)
- P1 pad 8: /GPIO14(TXD0) -> (no net)
